File: gardencore.brd (EAGLE design)
At the start: 91.4 x 30.5 mm, 14 parts, among them U1 tmp36

Commit message: logo labels and design rule check
Parts:
- removed U1: tmp36, SparkFun-Sensors:TO-92
- added R8: 10K, SparkFun-Passives:AXIAL-0.3
- added S1: (no value), SparkFun-Electromechanical:TACTILE-PTH
- added TEMP: LM50, linear:SOT23
- added U$1: (no value), SparkFun-Aesthetics:OSHW-LOGO-S
- moved LED2 12.8 mm to (22.9, 68.6)
- moved LED3 7.73 mm to (27.9, 68.6)
- moved R4 3.81 mm to (19.1, 53.3)
- moved LED1 2.84 mm to (17.8, 68.6)
- moved R5 2.54 mm to (22.9, 53.3)
- renumbered Q1 to NPN
Connections:
- net +3V3: now also S1.1, TEMP.1; no longer U1.1
- net A1: now also TEMP.2; no longer U1.2
- net D3: now also R8.P$2, S1.3
- net GND: now also R8.P$1, TEMP.3; no longer U1.3
Routing:
- net D3: track 0.00 -> 41.5 mm
- net D1: track 28.0 -> 15.9 mm
- net D2: track 30.6 -> 18.4 mm
- net GND: track 106.4 -> 118.2 mm, vias 0 -> 2
- net +3V3: track 128.9 -> 117.8 mm, vias 0 -> 1
- net N$5: track 21.9 -> 11.2 mm
- net D0: track 23.7 -> 13.3 mm
- net A1: track 73.9 -> 69.1 mm
- net N$6: track 13.5 -> 10.7 mm
- net N$4: track 12.5 -> 13.8 mm
- net A0: track 34.7 -> 33.9 mm
Other:
- board size 91.4 x 30.5 mm -> 91.4 x 31.1 mm
- board text added: "LED1"
- board text added: "LED2"
- board text added: "LED3"
- board text added: "NPN"
- board text added: "button"
- board text added: "photo"
- board text removed: "gardencore"
