File: gardencore.sch (EAGLE design)
At the start: 14 parts, among them U1 tmp36

Commit message: logo labels and design rule check
Parts:
- removed U1: tmp36, SparkFun-Sensors:TMP36GT9
- added R8: 10K, SparkFun-Passives:RESISTORAXIAL-0.3
- added S1: (no value), SparkFun-Electromechanical:TAC_SWITCHPTH
- added TEMP: LM50, linear:LM50
- renumbered Q1 to NPN
Connections:
- net +3V3: now also S1.1, TEMP.+VS; no longer U1.VCC
- net A1: now also TEMP.VO; no longer U1.VOUT
- net D3: now also R8.2, S1.3
- net GND: now also R8.1, TEMP.GND; no longer U1.GND
Other:
- moved on the sheet: LED1, LED2, LED3, R4, R5, R6
